File: Arrington 4 voice equivalent/Arrington 4 voice equivalent.kicad_pcb (KiCad board)
At the start: 2 copper layers, 55.8 x 40.1 mm, 18 parts, among them J1 SJ1-3525N, J2 DB25_Male, J3 RCJ-013, SW1 SW_SPDT, U1 74LS05

Commit message: start on rom pack and updates to sound PCBs
Parts:
- R6: value 72.5K -> 82.5K
Changed lines of the file:
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@@
     (property "PARTREV" "1.02")
     (property "STANDARD" "Manufacturer recommendation")
-    (property "Sheetfile" "Arrington 4 voice equivalent SMD.kicad_sch")
+    (property "Sheetfile" "Arrington 4 voice equivalent.kicad_sch")
     (property "Sheetname" "")
     (attr through_hole)
@@
     (property "PART_REV" "B")
     (property "STANDARD" "Manufacturer recommendations")
-    (property "Sheetfile" "Arrington 4 voice equivalent SMD.kicad_sch")
+    (property "Sheetfile" "Arrington 4 voice equivalent.kicad_sch")
     (property "Sheetname" "")
     (attr through_hole)
@@
       (effects (font (size 1 1) (thickness 0.15)))
     )
-    (fp_text value "72.5K" (at 5.08 -2.286 90) (layer "F.SilkS")
-      (effects (font (size 1 1) (thickness 0.15)))
-    )
+    (fp_text value "82.5K" (at 5.08 -2.286 90) (layer "F.SilkS")
+      (effects (font (size 1 1) (thickness 0.15)))
+    )
