File: Arrington 4 voice equivalent/Arrington 4 voice equivalent.kicad_sch (KiCad schematic)
At the start: 16 parts, among them J1 SJ1-3525N, J2 DB25_Male, SW1 SW_SPDT, U1 74LS05

Commit message: start on rom pack and updates to sound PCBs
Parts:
- R6: value 72.5K -> 82.5K
- gave numbers to parts that had none: 1
Changed lines of the file:
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@@
     (in_bom yes) (on_board yes) (fields_autoplaced)
     (property "Reference" "R6" (id 0) (at 128.905 75.0275 90))
-    (property "Value" "72.5K" (id 1) (at 128.905 77.8026 90))
+    (property "Value" "82.5K" (id 1) (at 128.905 77.8026 90))
     (property "Footprint" "Resistor_THT:R_Axial_DIN0207_L6.3mm_D2.5mm_P10.16mm_Horizontal" (id 2) (at 128.905 81.788 90)
       (effects (font (size 1.27 1.27)) hide)
@@
   (symbol (lib_id "Evan's misc parts:RCJ-013") (at 77.47 107.95 0) (mirror x) (unit 1)
     (in_bom yes) (on_board yes) (fields_autoplaced)
-    (property "Reference" "J?" (id 0) (at 73.533 107.0415 0)
+    (property "Reference" "J3" (id 0) (at 73.533 107.0415 0)
       (effects (font (size 1.27 1.27)) (justify right))
     )
@@
   (symbol (lib_id "power:GND") (at 85.09 110.49 0) (unit 1)
     (in_bom yes) (on_board yes) (fields_autoplaced)
-    (property "Reference" "#PWR?" (id 0) (at 85.09 116.84 0)
+    (property "Reference" "#PWR0101" (id 0) (at 85.09 116.84 0)
       (effects (font (size 1.27 1.27)) hide)
     )
@@
     )
     (path "/cacca2a5-ee01-47ed-b7f6-6cd97aa80a5e"
-      (reference "#PWR?") (unit 1) (value "GND") (footprint "")
+      (reference "#PWR0101") (unit 1) (value "GND") (footprint "")
     )
     (path "/a38425d6-86f5-471e-8b7f-240e2bbd0742"
@@
     )
     (path "/544e74c4-3ec3-4ef2-9ff1-d18c427a83b2"
-      (reference "J?") (unit 1) (value "RCJ-013") (footprint "CUI_RCJ-013")
+      (reference "J3") (unit 1) (value "RCJ-013") (footprint "CUI_RCJ-013")
     )
     (path "/c6e7158c-902b-4428-b0a1-86431224fa07"
@@
     )
     (path "/02233431-e289-43dc-8d58-45e22a9ff628"
-      (reference "R6") (unit 1) (value "72.5K") (footprint "Resistor_THT:R_Axial_DIN0207_L6.3mm_D2.5mm_P10.16mm_Horizontal")
+      (reference "R6") (unit 1) (value "82.5K") (footprint "Resistor_THT:R_Axial_DIN0207_L6.3mm_D2.5mm_P10.16mm_Horizontal")
     )
     (path "/ea95b2b2-ecc9-45b8-af1b-3ad9d4dab1a4"
