File: Arrington 4 voice equivalent SMD/Arrington 4 voice equivalent SMD.kicad_sch (KiCad schematic)
At the start: 19 parts, among them J1 SJ1-3525N, J2 DB25_Male, J3 RCJ-013, SW1 SW_SPDT, U1 74LS05, U2 74LS05

Commit message: start on rom pack and updates to sound PCBs
Parts:
- R6: value 72.5K -> 82.5K
Changed lines of the file:
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@@
     (in_bom yes) (on_board yes) (fields_autoplaced)
     (property "Reference" "R6" (id 0) (at 102.87 84.5525 90))
-    (property "Value" "72.5K" (id 1) (at 102.87 87.3276 90))
+    (property "Value" "82.5K" (id 1) (at 102.87 87.3276 90))
     (property "Footprint" "Resistor_SMD:R_0603_1608Metric" (id 2) (at 102.87 91.313 90)
       (effects (font (size 1.27 1.27)) hide)
@@
     )
     (path "/937939a7-3d48-498a-98b7-bb48d04ada01"
-      (reference "R6") (unit 1) (value "72.5K") (footprint "Resistor_SMD:R_0603_1608Metric")
+      (reference "R6") (unit 1) (value "82.5K") (footprint "Resistor_SMD:R_0603_1608Metric")
     )
     (path "/0a7da8e8-4a29-4619-8c2a-45042f49f661"
