File: Arrington 4 voice equivalent SMD/Arrington 4 voice equivalent SMD.kicad_pcb (KiCad board)
At the start: 2 copper layers, 31.8 x 40.1 mm, 21 parts, among them J1 SJ1-3525N, J2 DB25_Male, J3 RCJ-013, SW1 SW_SPDT, U1 74LS05, U2 74LS05

Commit message: start on rom pack and updates to sound PCBs
Parts:
- R6: value 72.5K -> 82.5K
Changed lines of the file:
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@@
   (net 34 "Net-(R8-Pad2)")
   (net 35 "Net-(SW1-Pad2)")
-  (net 36 "Net-(U2-Pad10)")
-  (net 37 "Net-(U2-Pad12)")
+  (net 36 "Net-(R10-Pad2)")
+  (net 37 "Net-(R11-Pad2)")
   (net 38 "unconnected-(U2-Pad2)")
   (net 39 "unconnected-(U2-Pad4)")
@@
       (effects (font (size 1 1) (thickness 0.15)))
     )
-    (fp_text value "72.5K" (at -3.81 0 90) (layer "F.SilkS")
+    (fp_text value "82.5K" (at -3.81 0 90) (layer "F.SilkS")
       (effects (font (size 1 1) (thickness 0.15)))
     )
@@
       (net 3 "/mixed audio") (pintype "passive"))
     (pad "2" smd roundrect locked (at 0.825 0 90) (size 0.8 0.95) (layers "B.Cu" "B.Paste" "B.Mask") (roundrect_rratio 0.25)
-      (net 36 "Net-(U2-Pad10)") (pintype "passive"))
+      (net 36 "Net-(R10-Pad2)") (pintype "passive"))
     (model "${KICAD6_3DMODEL_DIR}/Resistor_SMD.3dshapes/R_0603_1608Metric.wrl"
       (offset (xyz 0 0 0))
@@
       (net 3 "/mixed audio") (pintype "passive"))
     (pad "2" smd roundrect locked (at 0.825 0 90) (size 0.8 0.95) (layers "B.Cu" "B.Paste" "B.Mask") (roundrect_rratio 0.25)
-      (net 37 "Net-(U2-Pad12)") (pintype "passive"))
+      (net 37 "Net-(R11-Pad2)") (pintype "passive"))
     (model "${KICAD6_3DMODEL_DIR}/Resistor_SMD.3dshapes/R_0603_1608Metric.wrl"
       (offset (xyz 0 0 0))
@@
       (net 2 "GND") (pintype "input"))
     (pad "10" smd roundrect locked (at 2.475 -1.27 270) (size 1.95 0.6) (layers "B.Cu" "B.Paste" "B.Mask") (roundrect_rratio 0.25)
-      (net 36 "Net-(U2-Pad10)") (pintype "open_collector"))
+      (net 36 "Net-(R10-Pad2)") (pintype "open_collector"))
     (pad "11" smd roundrect locked (at 2.475 0 270) (size 1.95 0.6) (layers "B.Cu" "B.Paste" "B.Mask") (roundrect_rratio 0.25)
       (net 19 "/bit 0") (pintype "input"))
     (pad "12" smd roundrect locked (at 2.475 1.27 270) (size 1.95 0.6) (layers "B.Cu" "B.Paste" "B.Mask") (roundrect_rratio 0.25)
-      (net 37 "Net-(U2-Pad12)") (pintype "open_collector"))
+      (net 37 "Net-(R11-Pad2)") (pintype "open_collector"))
     (pad "13" smd roundrect locked (at 2.475 2.54 270) (size 1.95 0.6) (layers "B.Cu" "B.Paste" "B.Mask") (roundrect_rratio 0.25)
       (net 20 "/bit 1") (pintype "input"))
