File: Sorcerer Modern Rom Pack/Sorcerer Modern Rom Pack.kicad_sch (KiCad schematic)
At the start: 100 parts, among them J1 ROMRD15, J10 A11, J11 A13, J12 A12, J13 A, J14 A, J15 A, J16 A, J17 A, J18 C, J19 B, J2 A14, J20 A, J21 A, J22 A, J23 A, J24 A, J25 A, J26 A, J27 A, J28 Sorcerer Cart Slot, J29 0 ENABLE, J3 ROMRD15, J30 1 ENABLE, J31 4 ENABLE, J32 5 ENABLE, J33 1 PROM, J34 2 PROM, J35 A, J36 A, J37 A, J38 A, J39 A, J4 A12, J40 A, J41 A, J42 A, J43 A, J44 A, J45 A, J46 A, J47 A, J48 A, J49 A, J5 Conn_01x01, J50 A, J51 A, J52 A, J53 A, J54 A, J55 A, J56 A, J57 A, J58 A, J59 A, J6 Conn_01x01, J60 A, J61 A, J62 A, J63 A, J64 A, J65 A, J66 A, J67 A, J68 A, J69 RAM cut, J7 A, J8 A14, J9 A10, U1 2716, U2 2716, U3 2716, U4 2716, U5 74LS11, U6 74LS138

Commit message: tiny schematic change
Other:
- moved on the sheet: U?

Commit message: silk for bank switched ROM PCB
Parts:
- removed C10, C11, C6, C7, C9: 0.1uF, Capacitor_THT:C_Disc_D4.3mm_W1.9mm_P5.00mm, symbol Device:C
- removed C2, C5: 6.8uF, Capacitor_THT:CP_Radial_Tantal_D4.5mm_P5.00mm, symbol Device:C_Polarized
- removed J1, J3: ROMRD15, Connector_PinHeader_2.54mm:PinHeader_1x01_P2.54mm_Vertical, symbol Connector_Generic:Conn_01x01
- removed J10: A11, Connector_PinHeader_2.54mm:PinHeader_1x01_P2.54mm_Vertical, symbol Connector_Generic:Conn_01x01
- removed J11: A13, Connector_PinHeader_2.54mm:PinHeader_1x01_P2.54mm_Vertical, symbol Connector_Generic:Conn_01x01
- removed J12, J4: A12, Connector_PinHeader_2.54mm:PinHeader_1x01_P2.54mm_Vertical, symbol Connector_Generic:Conn_01x01
- removed J13, J14, J15, J16, J17, J20, J21, J22, J23, J24, J25, J26, J27, J35, J36, J37, J38, J39, J40, J41, J42, J43, J44, J45, J46, J47, J48, J49, J50, J51, J52, J53, J54, J55, J56, J57, J58, J59, J60, J61, J62, J63, J64, J65, J66, J67, J68, J7: A, Connector_PinHeader_2.54mm:PinHeader_1x01_P2.54mm_Vertical, symbol Connector_Generic:Conn_01x01
- removed J18: C, Connector_PinHeader_2.54mm:PinHeader_1x01_P2.54mm_Vertical, symbol Connector_Generic:Conn_01x01
- removed J19: B, Connector_PinHeader_2.54mm:PinHeader_1x01_P2.54mm_Vertical, symbol Connector_Generic:Conn_01x01
- removed J2, J8: A14, Connector_PinHeader_2.54mm:PinHeader_1x01_P2.54mm_Vertical, symbol Connector_Generic:Conn_01x01
- removed J29: 0 ENABLE, Connector_PinHeader_2.54mm:PinHeader_1x01_P2.54mm_Vertical, symbol Connector_Generic:Conn_01x01
- removed J30: 1 ENABLE, Connector_PinHeader_2.54mm:PinHeader_1x01_P2.54mm_Vertical, symbol Connector_Generic:Conn_01x01
- removed J31: 4 ENABLE, Connector_PinHeader_2.54mm:PinHeader_1x01_P2.54mm_Vertical, symbol Connector_Generic:Conn_01x01
- removed J32: 5 ENABLE, Connector_PinHeader_2.54mm:PinHeader_1x01_P2.54mm_Vertical, symbol Connector_Generic:Conn_01x01
- removed J33: 1 PROM, Connector_PinHeader_2.54mm:PinHeader_1x01_P2.54mm_Vertical, symbol Connector_Generic:Conn_01x01
- removed J34: 2 PROM, Connector_PinHeader_2.54mm:PinHeader_1x01_P2.54mm_Vertical, symbol Connector_Generic:Conn_01x01
- removed J5, J6: Conn_01x01, Connector_PinHeader_2.54mm:PinHeader_1x01_P2.54mm_Vertical, symbol Connector_Generic:Conn_01x01
- removed J69: RAM cut, Jumper:SolderJumper-2_P1.3mm_Open_RoundedPad1.0x1.5mm, symbol Connector_Generic:Conn_01x02
- removed J9: A10, Connector_PinHeader_2.54mm:PinHeader_1x01_P2.54mm_Vertical, symbol Connector_Generic:Conn_01x01
- removed SW?: SW_DIP_x06, symbol Switch:SW_DIP_x06
- removed U1, U2, U3, U4: 2716, Package_DIP:DIP-24_W15.24mm, symbol Evan's misc parts:2716
- removed U5: 74LS11, Package_DIP:DIP-14_W7.62mm, symbol 74xx:74LS11
- removed U6: 74LS138, Package_DIP:DIP-16_W7.62mm, symbol 74xx:74LS138
- added SW1: SW_DIP_x06, Button_Switch_THT:SW_DIP_SPSTx06_Piano_10.8x16.8mm_W7.62mm_P2.54mm, symbol Switch:SW_DIP_x06
- R1, R2, R3, R4, R5, R6, R7: renamed from R?; value R -> 4.7K; footprint (none) -> Resistor_THT:R_Axial_DIN0204_L3.6mm_D1.6mm_P1.90mm_Vertical
- U1, U2: renamed from U?; footprint (none) -> Package_DIP:DIP-16_W7.62mm
- gave numbers to parts that had none: 4
Connections:
- net GND: now also SW1.1, SW1.2, SW1.3, SW1.4, SW1.5, SW1.6
- net ROM14: now also SW1.8
- net ROM15: now also SW1.7
- net at R4.2, U1.1 (B3): now also SW1.9
- net at R3.2, U1.14 (B2): now also SW1.10
- net at R1.2, U1.9 (B0): now also SW1.12
- net at R2.2, U1.11 (B1): now also SW1.11
Other:
- note removed: "+12"
- note removed: "+5"
- note removed: "-5"
- note removed: "0 ENABLE"
- note removed: "1"
- note removed: "1 ENABLE"
- note removed: "18"
- note removed: "19"
- note removed: "2"
- note removed: "2 ENABLE"
- note removed: "20"
- note removed: "21"
- note removed: "3"
- note removed: "3 ENABLE"
- note removed: "4"
- note removed: "5A"
- note removed: "5B"
- note removed: "6"
- note removed: "7"
- note removed: "A"
- note removed: "A10"
- note removed: "A11"
- note removed: "B"
- note removed: "C"
- note removed: "D"
- note removed: "E"
- note removed: "F"
- note removed: "G"
- note removed: "Gnd"
- note removed: "ROM 1"
- note removed: "ROM 2"
- note removed: "ROM 3"
- note removed: "ROM 4"
- moved on the sheet: C1, C3, C4, C8, D1, D2, D3, J28, R1, R2, R3, R4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
