File: s100 expansion chassis/S100 connectors.kicad_sch (KiCad schematic)
At the start: 6 parts, among them J5 346-100-520-802, J6 346-100-520-802, J7 346-100-520-802, J8 346-100-520-802, J9 346-100-520-802

Commit message: cleaned up things
Parts:
- J1, J2: renamed from J5; footprint Evan's misc parts:346100520802 -> Evan's parts:346100520802
- J5: renamed from J8; footprint Evan's misc parts:346100520802 -> Evan's parts:346100520802
- J6: renamed from J9; footprint Evan's misc parts:346100520802 -> Evan's parts:346100520802
- J7: renamed from J6; footprint Evan's misc parts:346100520802 -> Evan's parts:346100520802
- J8: renamed from J7; footprint Evan's misc parts:346100520802 -> Evan's parts:346100520802
Changed lines of the file:
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@@
   (symbol (lib_name "346-100-520-802_1") (lib_id "Evan's misc parts:346-100-520-802") (at 60.325 24.13 0) (unit 1)
     (in_bom yes) (on_board yes) (dnp no) (fields_autoplaced)
-    (property "Reference" "J5" (at 73.025 17.6743 0)
+    (property "Reference" "J2" (at 73.025 17.6743 0)
       (effects (font (size 1.27 1.27)))
     )
@@
       (effects (font (size 1.27 1.27)))
     )
-    (property "Footprint" "Evan's misc parts:346100520802" (at 81.915 21.59 0)
+    (property "Footprint" "Evan's parts:346100520802" (at 81.915 21.59 0)
       (effects (font (size 1.27 1.27)) (justify left) hide)
     )
@@
   (symbol (lib_name "346-100-520-802_1") (lib_id "Evan's misc parts:346-100-520-802") (at 135.89 24.13 0) (unit 1)
     (in_bom yes) (on_board yes) (dnp no) (fields_autoplaced)
-    (property "Reference" "J7" (at 148.59 18.6309 0)
+    (property "Reference" "J8" (at 148.59 18.6309 0)
       (effects (font (size 1.27 1.27)))
     )
@@
       (effects (font (size 1.27 1.27)))
     )
-    (property "Footprint" "Evan's misc parts:346100520802" (at 157.48 21.59 0)
+    (property "Footprint" "Evan's parts:346100520802" (at 157.48 21.59 0)
       (effects (font (size 1.27 1.27)) (justify left) hide)
     )
@@
   (symbol (lib_name "346-100-520-802_1") (lib_id "Evan's misc parts:346-100-520-802") (at 173.99 24.13 0) (unit 1)
     (in_bom yes) (on_board yes) (dnp no) (fields_autoplaced)
-    (property "Reference" "J8" (at 186.69 17.6743 0)
+    (property "Reference" "J5" (at 186.69 17.6743 0)
       (effects (font (size 1.27 1.27)))
     )
@@
       (effects (font (size 1.27 1.27)))
     )
-    (property "Footprint" "Evan's misc parts:346100520802" (at 195.58 21.59 0)
+    (property "Footprint" "Evan's parts:346100520802" (at 195.58 21.59 0)
       (effects (font (size 1.27 1.27)) (justify left) hide)
     )
@@
   (symbol (lib_name "346-100-520-802_1") (lib_id "Evan's misc parts:346-100-520-802") (at 98.425 24.13 0) (unit 1)
     (in_bom yes) (on_board yes) (dnp no) (fields_autoplaced)
-    (property "Reference" "J6" (at 111.125 18.6309 0)
+    (property "Reference" "J7" (at 111.125 18.6309 0)
       (effects (font (size 1.27 1.27)))
     )
@@
       (effects (font (size 1.27 1.27)))
     )
-    (property "Footprint" "Evan's misc parts:346100520802" (at 120.015 21.59 0)
+    (property "Footprint" "Evan's parts:346100520802" (at 120.015 21.59 0)
       (effects (font (size 1.27 1.27)) (justify left) hide)
     )
@@
   (symbol (lib_name "346-100-520-802_1") (lib_id "Evan's misc parts:346-100-520-802") (at 21.59 24.13 0) (unit 1)
     (in_bom yes) (on_board yes) (dnp no) (fields_autoplaced)
-    (property "Reference" "J5" (at 34.29 17.6743 0)
+    (property "Reference" "J1" (at 34.29 17.6743 0)
       (effects (font (size 1.27 1.27)))
     )
@@
       (effects (font (size 1.27 1.27)))
     )
-    (property "Footprint" "Evan's misc parts:346100520802" (at 43.18 21.59 0)
+    (property "Footprint" "Evan's parts:346100520802" (at 43.18 21.59 0)
       (effects (font (size 1.27 1.27)) (justify left) hide)
     )
@@
   (symbol (lib_name "346-100-520-802_1") (lib_id "Evan's misc parts:346-100-520-802") (at 215.9 24.13 0) (unit 1)
     (in_bom yes) (on_board yes) (dnp no) (fields_autoplaced)
-    (property "Reference" "J9" (at 228.6 17.6743 0)
+    (property "Reference" "J6" (at 228.6 17.6743 0)
       (effects (font (size 1.27 1.27)))
     )
@@
       (effects (font (size 1.27 1.27)))
     )
-    (property "Footprint" "Evan's misc parts:346100520802" (at 237.49 21.59 0)
-      (effects (font (size 1.27 1.27)) (justify left) hide)
-    )
+    (property "Footprint" "Evan's parts:346100520802" (at 237.49 21.59 0)
+      (effects (font (size 1.27 1.27)) (justify left) hide)
+    )
