File: s100 expansion chassis/s100 expansion chassis.kicad_sch (KiCad schematic)
At the start: 73 parts, among them J1 Power In, J3 Sorcerer ribbon, U1 74LS241, U10 DP8304BN, U11 DP8304BN, U12 DP8304BN, U13 74LS32, U14 74LS08, U15 74LS02, U16 74LS04, U17 6331 PROM, U18 74LS74, U19 74LS02, U2 74LS241, U20 74LS04, U21 74LS00, U22 74LS08, U23 74LS10, U3 74LS241, U4 74LS241, U5 74LS241, U6 74LS241, U7 74LS241, U8 74LS241, U9 DP8304BN, Y1 2Mhz

Commit message: tweaks to schematic
Parts:
- removed R10, R11, R12: 2.2K, symbol Device:R
- added R19, R20, R21: 2.2K, symbol Device:R
- J3: footprint (none) -> Connector_PinHeader_2.54mm:PinHeader_2x25_P2.54mm_Vertical
Connections:
- net +5V: now also R19.1, R20.1, R21.1
- net at U4.19 (OEb): now also R20.2
- net at U7.6 (I2a): now also R19.2
- net at U18.10 (~{S}): now also R21.2
Changed lines of the file:
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@@
     )
   )
+  (symbol (lib_id "Device:R") (at 276.86 148.59 90) (unit 1)
+    (in_bom yes) (on_board yes) (dnp no)
+    (property "Reference" "R21" (at 277.495 150.495 90)
+      (effects (font (size 1.27 1.27)) (justify left))
+    )
+    (property "Value" "2.2K" (at 278.765 146.685 90)
+      (effects (font (size 1.27 1.27)) (justify left))
+    )
+    (property "Footprint" "" (at 276.86 150.368 90)
+      (effects (font (size 1.27 1.27)) hide)
+    )
+    (property "Datasheet" "~" (at 276.86 148.59 0)
+      (effects (font (size 1.27 1.27)) hide)
+    )
+    (pin "1")
+    (pin "2")
+    (instances
+      (project "s100 expansion chassis"
+        (path "/aa27471d-b1e6-44de-bc58-907b9dc0c658"
+          (reference "R21") (unit 1)
+        )
+      )
+    )
+  )
   (symbol (lib_id "power:GND") (at 434.34 69.85 0) (unit 1)
     (in_bom yes) (on_board yes) (dnp no) (fields_autoplaced)
@@
     )
   )
+  (symbol (lib_id "Device:R") (at 347.98 215.9 90) (unit 1)
+    (in_bom yes) (on_board yes) (dnp no)
+    (property "Reference" "R19" (at 348.615 217.805 90)
+      (effects (font (size 1.27 1.27)) (justify left))
+    )
+    (property "Value" "2.2K" (at 349.885 213.995 90)
+      (effects (font (size 1.27 1.27)) (justify left))
+    )
+    (property "Footprint" "" (at 347.98 217.678 90)
+      (effects (font (size 1.27 1.27)) hide)
+    )
+    (property "Datasheet" "~" (at 347.98 215.9 0)
+      (effects (font (size 1.27 1.27)) hide)
+    )
+    (pin "1")
+    (pin "2")
+    (instances
+      (project "s100 expansion chassis"
+        (path "/aa27471d-b1e6-44de-bc58-907b9dc0c658"
+          (reference "R19") (unit 1)
+        )
+      )
+    )
+  )
   (symbol (lib_id "74xx:74LS04") (at 334.01 34.29 0) (unit 7)
     (in_bom yes) (on_board yes) (dnp no) (fields_autoplaced)
@@
     )
   )
-  (symbol (lib_id "Device:R") (at 276.86 148.59 90) (unit 1)
-    (in_bom yes) (on_board yes) (dnp no)
-    (property "Reference" "R12" (at 277.495 150.495 90)
-      (effects (font (size 1.27 1.27)) (justify left))
-    )
-    (property "Value" "2.2K" (at 278.765 146.685 90)
-      (effects (font (size 1.27 1.27)) (justify left))
-    )
-    (property "Footprint" "" (at 276.86 150.368 90)
-      (effects (font (size 1.27 1.27)) hide)
-    )
-    (property "Datasheet" "~" (at 276.86 148.59 0)
-      (effects (font (size 1.27 1.27)) hide)
-    )
-    (pin "1")
-    (pin "2")
-    (instances
-      (project "s100 expansion chassis"
-        (path "/aa27471d-b1e6-44de-bc58-907b9dc0c658"
-          (reference "R12") (unit 1)
-        )
-      )
-    )
-  )
   (symbol (lib_id "power:GND") (at 361.95 69.85 0) (unit 1)
     (in_bom yes) (on_board yes) (dnp no) (fields_autoplaced)
@@
     )
   )
-  (symbol (lib_id "Device:R") (at 174.625 117.475 270) (mirror x) (unit 1)
-    (in_bom yes) (on_board yes) (dnp no)
-    (property "Reference" "R11" (at 173.99 119.38 90)
-      (effects (font (size 1.27 1.27)) (justify left))
-    )
-    (property "Value" "2.2K" (at 172.72 115.57 90)
-      (effects (font (size 1.27 1.27)) (justify left))
-    )
-    (property "Footprint" "" (at 174.625 119.253 90)
-      (effects (font (size 1.27 1.27)) hide)
-    )
-    (property "Datasheet" "~" (at 174.625 117.475 0)
-      (effects (font (size 1.27 1.27)) hide)
-    )
-    (pin "1")
-    (pin "2")
-    (instances
-      (project "s100 expansion chassis"
-        (path "/aa27471d-b1e6-44de-bc58-907b9dc0c658"
-          (reference "R11") (unit 1)
-        )
-      )
-    )
-  )
   (symbol (lib_id "Device:R") (at 241.3 249.555 0) (unit 1)
     (in_bom yes) (on_board yes) (dnp no) (fields_autoplaced)
@@
       (effects (font (size 1.27 1.27)))
     )
-    (property "Footprint" "" (at 396.24 374.65 0)
+    (property "Footprint" "Connector_PinHeader_2.54mm:PinHeader_2x25_P2.54mm_Vertical" (at 396.24 374.65 0)
       (effects (font (size 1.27 1.27)) hide)
     )
@@
     )
   )
+  (symbol (lib_id "Device:R") (at 174.625 117.475 270) (mirror x) (unit 1)
+    (in_bom yes) (on_board yes) (dnp no)
+    (property "Reference" "R20" (at 173.99 119.38 90)
+      (effects (font (size 1.27 1.27)) (justify left))
+    )
+    (property "Value" "2.2K" (at 172.72 115.57 90)
+      (effects (font (size 1.27 1.27)) (justify left))
+    )
+    (property "Footprint" "" (at 174.625 119.253 90)
+      (effects (font (size 1.27 1.27)) hide)
+    )
+    (property "Datasheet" "~" (at 174.625 117.475 0)
+      (effects (font (size 1.27 1.27)) hide)
+    )
+    (pin "1")
+    (pin "2")
+    (instances
+      (project "s100 expansion chassis"
+        (path "/aa27471d-b1e6-44de-bc58-907b9dc0c658"
+          (reference "R20") (unit 1)
+        )
+      )
+    )
+  )
   (symbol (lib_id "74xx:74LS04") (at 297.815 243.84 0) (unit 4)
     (in_bom yes) (on_board yes) (dnp no)
@@
         )
       )
-    )
-  )
-  (symbol (lib_id "Device:R") (at 347.98 215.9 90) (unit 1)
-    (in_bom yes) (on_board yes) (dnp no)
-    (property "Reference" "R10" (at 348.615 217.805 90)
-      (effects (font (size 1.27 1.27)) (justify left))
-    )
-    (property "Value" "2.2K" (at 349.885 213.995 90)
-      (effects (font (size 1.27 1.27)) (justify left))
-    )
-    (property "Footprint" "" (at 347.98 217.678 90)
-      (effects (font (size 1.27 1.27)) hide)
-    )
-    (property "Datasheet" "~" (at 347.98 215.9 0)
-      (effects (font (size 1.27 1.27)) hide)
-    )
-    (pin "1")
-    (pin "2")
-    (instances
-      (project "s100 expansion chassis"
-        (path "/aa27471d-b1e6-44de-bc58-907b9dc0c658"
-          (reference "R10") (unit 1)
-        )
-      )

Commit message: cleaned up things
Parts:
- C1, C2: footprint (none) -> Capacitor_THT:CP_Radial_Tantal_D8.0mm_P5.00mm
- C10, C11, C12, C13, C14, C15, C16, C18, C19, C3, C4, C5, C6, C7, C8, C9: footprint (none) -> Evan's parts:C_Disc_D6.0mm_W2.5mm_P6.35mm
- C3: footprint Evan's misc parts:CP_Radial_D35.0mm_P12.90mm_SnapIn -> Evan's parts:CP_Radial_D35.0mm_P12.90mm_SnapIn
- J1: footprint Evan's misc parts:5 pin inline molex 0.93 -> Evan's parts:5 pin inline molex 0.93
- R1, R10, R11, R12, R13, R14, R15, R16, R17, R18, R19, R2, R20, R21, R3, R4, R5, R6, R7, R8, R9: footprint (none) -> Evan's parts:R_Axial_DIN0204_L3.6mm_D1.6mm_P12.7mm_Horizontal
- U1, U10, U11, U12, U2, U3, U4, U5, U6, U7, U8, U9: footprint (none) -> Package_DIP:DIP-20_W7.62mm
- U13, U14, U15, U16, U18, U19, U20, U21, U22, U23: footprint (none) -> Package_DIP:DIP-14_W7.62mm
- Y1: footprint (none) -> Crystal:Crystal_HC33-U_Horizontal
